File: Rev A/mini project newest.sch (KiCad schematic (older format))
At the start: 26 parts, among them J1 Conn_01x02, Q1 Q_NMOS_DSG, U1 LM555, U2 LM555

Commit message: new foot prints, new traces, new coat of paint. a few errors still need to be worked out, mostly with footprints not playing well with thicc traces
Parts:
- U1, U2: symbol Timer:LM555 -> mini-project-newest-rescue:LM555-Timer
Changed lines of the file:
@@
 	8600 2250 8950 2250
 $Comp
-L Timer:LM555 U1
+L mini-project-newest-rescue:LM555-Timer U1
 U 1 1 5F77AB9D
 P 2900 2600
@@
 $EndComp
 $Comp
-L Timer:LM555 U2
+L mini-project-newest-rescue:LM555-Timer U2
 U 1 1 5F787D1A
 P 5800 2600

Commit message: fixed mosfet footprint, made vias bigger, going to clean up traces
Parts:
- removed Q1: Q_NMOS_DSG, Package_TO_SOT_THT:TO-92, symbol Device:Q_NMOS_DSG
- added Q1: Q_NMOS_SGD, Package_TO_SOT_THT:TO-92, symbol Device:Q_NMOS_SGD
Connections:
- net Earth: now also Q1.1 (S)
- net at C4.2, R3.2, TP7.1: now also Q1.3 (D)
- net at TP5.1, U2.3 (Q): now also Q1.2 (G)
Changed lines of the file:
@@
 EESchema Schematic File Version 4
+LIBS:mini project newest-cache
 EELAYER 30 0
 EELAYER END
@@
 R3 Current Measure
 $Comp
-L Device:Q_NMOS_DSG Q1
-U 1 1 5F7DE7DE
+L Device:Q_NMOS_SGD Q1
+U 1 1 5F77F761
 P 7525 2400
 F 0 "Q1" H 7731 2446 50  0000 L CNN
-F 1 "Q_NMOS_DSG" H 7731 2355 50  0000 L CNN
+F 1 "Q_NMOS_SGD" H 7731 2355 50  0000 L CNN
 F 2 "Package_TO_SOT_THT:TO-92" H 7725 2500 50  0001 C CNN
 F 3 "~" H 7525 2400 50  0001 C CNN

Commit message: Fixed traces not grounding properly, fixed pad too close to pad bugs, finished silkscreen, changed mounting hole sizes, repositioned TPs
Connections:
- net GND is gone; now on net Earth: J1.2 (Pin_2), TP1.1, TP2.1, TP3.1
Changed lines of the file:
@@
 EESchema Schematic File Version 4
-LIBS:mini project newest-cache
 EELAYER 30 0
 EELAYER END
@@
 Speaker
 Wire Wire Line
-	8675 2350 9775 2350
-Wire Wire Line
 	8675 2350 8675 6000
 Wire Wire Line
@@
 	1    0    0    -1
 $EndComp
-$Comp
-L power:GND #PWR0102
-U 1 1 5F7B091D
-P 9100 1425
-F 0 "#PWR0102" H 9100 1175 50  0001 C CNN
-F 1 "GND" H 9105 1252 50  0000 C CNN
-F 2 "" H 9100 1425 50  0001 C CNN
-F 3 "" H 9100 1425 50  0001 C CNN
-	1    9100 1425
-	1    0    0    -1
-$EndComp
-Wire Wire Line
-	9100 1425 9100 1300
 $Comp
 L Connector:TestPoint TP4
@@
 	1    0    0    -1
 $EndComp
-$Comp
-L power:GND #PWR0103
-U 1 1 5F7C07AF
-P 2025 6900
-F 0 "#PWR0103" H 2025 6650 50  0001 C CNN
-F 1 "GND" H 2030 6727 50  0000 C CNN
-F 2 "" H 2025 6900 50  0001 C CNN
-F 3 "" H 2025 6900 50  0001 C CNN
-	1    2025 6900
-	1    0    0    -1
-$EndComp
-$Comp
-L power:GND #PWR0104
-U 1 1 5F7C1724
-P 2625 6900
-F 0 "#PWR0104" H 2625 6650 50  0001 C CNN
-F 1 "GND" H 2630 6727 50  0000 C CNN
-F 2 "" H 2625 6900 50  0001 C CNN
-F 3 "" H 2625 6900 50  0001 C CNN
-	1    2625 6900
-	1    0    0    -1
-$EndComp
-$Comp
-L power:GND #PWR0105
-U 1 1 5F7C40C3
-P 3200 6900
-F 0 "#PWR0105" H 3200 6650 50  0001 C CNN
-F 1 "GND" H 3205 6727 50  0000 C CNN
-F 2 "" H 3200 6900 50  0001 C CNN
-F 3 "" H 3200 6900 50  0001 C CNN
-	1    3200 6900
-	1    0    0    -1
-$EndComp
 Wire Wire Line
 	2025 6625 2025 6900
@@
 	1    0    0    -1
 $EndComp
+Wire Wire Line
+	8675 2350 9775 2350
+$Comp
+L power:Earth #PWR?
+U 1 1 5F78CD2D
+P 9100 1375
+F 0 "#PWR?" H 9100 1125 50  0001 C CNN
+F 1 "Earth" H 9100 1225 50  0001 C CNN
+F 2 "" H 9100 1375 50  0001 C CNN
+F 3 "~" H 9100 1375 50  0001 C CNN
+	1    9100 1375
+	1    0    0    -1
+$EndComp
+Wire Wire Line
+	9100 1300 9100 1375
+$Comp
+L power:Earth #PWR?
+U 1 1 5F7924F0
+P 2025 6900
+F 0 "#PWR?" H 2025 6650 50  0001 C CNN
+F 1 "Earth" H 2025 6750 50  0001 C CNN
+F 2 "" H 2025 6900 50  0001 C CNN
+F 3 "~" H 2025 6900 50  0001 C CNN
+	1    2025 6900
+	1    0    0    -1
+$EndComp
+$Comp
+L power:Earth #PWR?
+U 1 1 5F795194
+P 2625 6900
+F 0 "#PWR?" H 2625 6650 50  0001 C CNN
+F 1 "Earth" H 2625 6750 50  0001 C CNN
+F 2 "" H 2625 6900 50  0001 C CNN
+F 3 "~" H 2625 6900 50  0001 C CNN
+	1    2625 6900
+	1    0    0    -1
+$EndComp
+$Comp
+L power:Earth #PWR?
+U 1 1 5F797EB9
+P 3200 6900
+F 0 "#PWR?" H 3200 6650 50  0001 C CNN
+F 1 "Earth" H 3200 6750 50  0001 C CNN
+F 2 "" H 3200 6900 50  0001 C CNN
+F 3 "~" H 3200 6900 50  0001 C CNN
+	1    3200 6900
+	1    0    0    -1
+$EndComp
